File: hardware/multiplexer_adc.kicad_sch (KiCad schematic)
At the start: 6 parts, among them P1 10k, P2 10k, P3 10k, P4 10k, U2 CD4051B

Commit message: Finalized first schematic version
Parts:
- removed P1, P2, P3, P4: 10k, Resistor_THT:R_Array_SIP4, symbol Device:R_Potentiometer
- renumbered C3 to C12, U2 to U3
