File: hardware/palmer_drum.kicad_sch (KiCad schematic)
At the start: 13 parts, among them J1 EURO_PWR, J2 SERGE_PWR, U3 L7805

Commit message: Finalized first schematic version
Parts:
- added J3, J4, J5, J6: Conn_02x05_Odd_Even, symbol Connector_Generic:Conn_02x05_Odd_Even
- renumbered C6 to C1, C7 to C2, C2 to C3, C1 to C4, C4 to C6, U3 to U1
Connections:
- net GND: now also J3.10 (Pin_10), J3.9 (Pin_9), J4.10 (Pin_10), J4.9 (Pin_9), J5.10 (Pin_10), J5.9 (Pin_9), J6.10 (Pin_10), J6.9 (Pin_9)
- new net +3V3: J3.7 (Pin_7), J3.8 (Pin_8), J4.7 (Pin_7), J4.8 (Pin_8), J5.7 (Pin_7), J5.8 (Pin_8), J6.7 (Pin_7), J6.8 (Pin_8)
- new net ADC_0_CONN_F: J4.1 (Pin_1)
- new net ADC_0_CONN_M: J6.1 (Pin_1)
- new net ADC_1_CONN_F: J4.2 (Pin_2)
- new net ADC_1_CONN_M: J6.2 (Pin_2)
- new net ADC_2_CONN_F: J4.3 (Pin_3)
- new net ADC_2_CONN_M: J6.3 (Pin_3)
- new net ADC_3_CONN_F: J4.4 (Pin_4)
- new net ADC_3_CONN_M: J6.4 (Pin_4)
- new net AUDIO_OUT_CONN_F: J3.6 (Pin_6)
- new net AUDIO_OUT_CONN_M: J5.6 (Pin_6)
- new net BTN_CONN_F: J4.6 (Pin_6)
- new net BTN_CONN_M: J6.6 (Pin_6)
- new net INPUT_CONN_F: J4.5 (Pin_5)
- new net INPUT_CONN_M: J6.5 (Pin_5)
- new net LED_1_CONN_F: J3.1 (Pin_1)
- new net LED_1_CONN_M: J5.1 (Pin_1)
- new net LED_2_CONN_F: J3.2 (Pin_2)
- new net LED_2_CONN_M: J5.2 (Pin_2)
- new net LED_3_CONN_F: J3.3 (Pin_3)
- new net LED_3_CONN_M: J5.3 (Pin_3)
- new net LED_4_CONN_F: J3.4 (Pin_4)
- new net LED_4_CONN_M: J5.4 (Pin_4)
- new net LED_PWM_CTRL_CONN_F: J3.5 (Pin_5)
- new net LED_PWM_CTRL_CONN_M: J5.5 (Pin_5)
Other:
- sheet INPUT_OUTPUT ports: added AUDIO_OUT_F, X_0_F, X_1_F, X_2_F, X_3_F; removed none
- sheet MCU ports: added PWM_AUDIO_OUT; removed none
- sheet MULTIPLEXER_ADC ports: added X_0, X_1, X_2, X_3; removed none

Commit message: Missing aop supply, fixed minor issues
Parts:
- added U2: TL072, symbol Amplifier_Operational:TL072
Connections:
- net +12V: now also U2.8 (V+)
- net -12V: now also U2.4 (V-)
Changed lines of the file:
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@@
 	)
 	(junction
+		(at 96.52 147.32)
+		(diameter 0)
+		(color 0 0 0 0)
+	)
+	(junction
 		(at 38.1 149.86)
 		(diameter 0)
@@
 	)
 	(junction
+		(at 96.52 170.18)
+		(diameter 0)
+		(color 0 0 0 0)
+	)
+	(junction
 		(at 53.34 147.32)
 		(diameter 0)
@@
 	(wire
 		(pts
+			(xy 111.76 170.18) (xy 96.52 170.18)
+		)
+		(stroke
+			(width 0)
+			(type default)
+		)
+	)
+	(wire
+		(pts
 			(xy 81.28 35.56) (xy 83.82 35.56)
 		)
@@
 	(wire
 		(pts
+			(xy 111.76 166.37) (xy 111.76 170.18)
+		)
+		(stroke
+			(width 0)
+			(type default)
+		)
+	)
+	(wire
+		(pts
 			(xy 140.97 115.57) (xy 140.97 119.38)
 		)
@@
 	(wire
 		(pts
+			(xy 111.76 151.13) (xy 111.76 147.32)
+		)
+		(stroke
+			(width 0)
+			(type default)
+		)
+	)
+	(wire
+		(pts
 			(xy 132.08 149.86) (xy 140.97 149.86)
 		)
@@
 	(wire
 		(pts
+			(xy 111.76 147.32) (xy 96.52 147.32)
+		)
+		(stroke
+			(width 0)
+			(type default)
+		)
+	)
+	(wire
+		(pts
 			(xy 45.72 184.15) (xy 45.72 182.88)
 		)
@@
 				)
 			)
+		)
+	)
+	(symbol
+		(lib_id "Amplifier_Operational:TL072")
+		(at 114.3 158.75 0)
+		(unit 3)
+		(body_style 1)
+		(exclude_from_sim no)
+		(in_bom yes)
+		(on_board yes)
+		(in_pos_files yes)
+		(dnp no)
+		(fields_autoplaced yes)
+		(property "Reference" "U2"
+			(at 113.03 157.4799 0)
+			(show_name no)
+			(do_not_autoplace no)
+			(effects
+				(font
+					(size 1.27 1.27)
+				)
+				(justify left)
+			)
+		)
+		(property "Value" "TL072"
+			(at 113.03 160.0199 0)
+			(show_name no)
+			(do_not_autoplace no)
+			(effects
+				(font
+					(size 1.27 1.27)
+				)
+				(justify left)
+			)
+		)
+		(property "Footprint" ""
+			(at 114.3 158.75 0)
+			(hide yes)
+			(show_name no)
+			(do_not_autoplace no)
+			(effects
+				(font
+					(size 1.27 1.27)
+				)
+			)
+		)
+		(property "Datasheet" "http://www.ti.com/lit/ds/symlink/tl071.pdf"
+			(at 114.3 158.75 0)
+			(hide yes)
+			(show_name no)
+			(do_not_autoplace no)
+			(effects
+				(font
+					(size 1.27 1.27)
+				)
+			)
+		)
+		(property "Description" "Dual Low-Noise JFET-Input Operational Amplifiers, DIP-8/SOIC-8"
+			(at 114.3 158.75 0)
+			(hide yes)
+			(show_name no)
+			(do_not_autoplace no)
+			(effects
+				(font
+					(size 1.27 1.27)
+				)
+			)
+		)
+		(pin "6"
+		)
+		(pin "7"
+		)
+		(pin "2"
+		)
+		(pin "5"
+		)
+		(pin "1"
+		)
+		(pin "3"
+		)
+		(pin "8"
+		)
+		(pin "4"
+		)
+		(instances
+			(project "palmer_drum"
+				(path "/a1c8c82f-599d-4a64-8030-47d97f65a492"
+					(reference "U2")
+					(unit 3)
+				)
+			)
